File: pcb/inz.kicad_sch (KiCad schematic)
At the start: 410 parts, among them U1 AMS1117-3.3, U2 ESP32-S3-WROOM-1

Commit message: pcb update
Connections:
- net at U62.1 (CLO): now also U63.3 (CLI); no longer U82.3 (CLI)
- net at U62.4 (DAO): now also U63.6 (DAI); no longer U82.6 (DAI)
- net at U187.1 (CLO): now also U188.3 (CLI); no longer U186.3 (CLI)
- net at U187.3 (CLI): now also U186.1 (CLO); no longer U188.1 (CLO)
- net at U187.4 (DAO): now also U188.6 (DAI); no longer U186.6 (DAI)
- net at U187.6 (DAI): now also U186.4 (DAO); no longer U188.4 (DAO)
- net at U232.1 (CLO): now also U233.3 (CLI); no longer U231.3 (CLI)
- net at U232.3 (CLI): now also U231.1 (CLO); no longer U233.1 (CLO)
- net at U232.4 (DAO): now also U233.6 (DAI); no longer U231.6 (DAI)
- net at U232.6 (DAI): now also U231.4 (DAO); no longer U233.4 (DAO)
- net at U228.1 (CLO): now also U229.3 (CLI); no longer U227.3 (CLI)
- net at U228.3 (CLI): now also U227.1 (CLO); no longer U229.1 (CLO)
- net at U228.4 (DAO): now also U229.6 (DAI); no longer U227.6 (DAI)
- net at U228.6 (DAI): now also U227.4 (DAO); no longer U229.4 (DAO)
- net at U391.1 (CLO): now also U392.3 (CLI); no longer U390.3 (CLI)
- net at U391.3 (CLI): now also U390.1 (CLO); no longer U392.1 (CLO)
- net at U391.4 (DAO): now also U392.6 (DAI); no longer U390.6 (DAI)
- net at U391.6 (DAI): now also U390.4 (DAO); no longer U392.4 (DAO)
- net at U29.1 (CLO): now also U30.3 (CLI); no longer U28.3 (CLI)
- net at U29.3 (CLI): now also U28.1 (CLO); no longer U30.1 (CLO)
- net at U29.4 (DAO): now also U30.6 (DAI); no longer U28.6 (DAI)
- net at U29.6 (DAI): now also U28.4 (DAO); no longer U30.4 (DAO)
- net at U322.1 (CLO): now also U323.3 (CLI); no longer U321.3 (CLI)
- net at U322.3 (CLI): now also U321.1 (CLO); no longer U302.1 (CLO)
- net at U322.4 (DAO): now also U323.6 (DAI); no longer U321.6 (DAI)
- net at U322.6 (DAI): now also U321.4 (DAO); no longer U302.4 (DAO)
- net at U305.1 (CLO): now also U306.3 (CLI); no longer U304.3 (CLI)
- net at U305.3 (CLI): now also U304.1 (CLO); no longer U306.1 (CLO)
- net at U305.4 (DAO): now also U306.6 (DAI); no longer U304.6 (DAI)
- net at U305.6 (DAI): now also U304.4 (DAO); no longer U306.4 (DAO)
- net at U396.1 (CLO): now also U397.3 (CLI); no longer U395.3 (CLI)
- net at U396.3 (CLI): now also U395.1 (CLO); no longer U397.1 (CLO)
- net at U396.4 (DAO): now also U397.6 (DAI); no longer U395.6 (DAI)
- net at U396.6 (DAI): now also U395.4 (DAO); no longer U397.4 (DAO)
- net at U78.1 (CLO): now also U79.3 (CLI); no longer U77.3 (CLI)
- net at U78.3 (CLI): now also U77.1 (CLO); no longer U79.1 (CLO)
- net at U78.4 (DAO): now also U79.6 (DAI); no longer U77.6 (DAI)
- net at U78.6 (DAI): now also U77.4 (DAO); no longer U79.4 (DAO)
- net at U81.1 (CLO): now also U82.3 (CLI); no longer U80.3 (CLI)
- net at U81.3 (CLI): now also U80.1 (CLO); no longer U82.1 (CLO)
- net at U81.4 (DAO): now also U82.6 (DAI); no longer U80.6 (DAI)
- net at U81.6 (DAI): now also U80.4 (DAO); no longer U82.4 (DAO)
- net at U225.1 (CLO): now also U226.3 (CLI); no longer U224.3 (CLI)
- net at U225.3 (CLI): now also U224.1 (CLO); no longer U226.1 (CLO)
- net at U225.4 (DAO): now also U226.6 (DAI); no longer U224.6 (DAI)
- net at U225.6 (DAI): now also U224.4 (DAO); no longer U226.4 (DAO)
- net at U383.1 (CLO): now also U384.3 (CLI)
- net at U383.3 (CLI): now also U382.1 (CLO); no longer U384.1 (CLO)
- net at U383.4 (DAO): now also U384.6 (DAI)
- net at U383.6 (DAI): now also U382.4 (DAO); no longer U384.4 (DAO)
- net at U105.1 (CLO): now also U106.3 (CLI); no longer U104.3 (CLI)
- net at U105.3 (CLI): now also U104.1 (CLO); no longer U106.1 (CLO)
- net at U105.4 (DAO): now also U106.6 (DAI); no longer U104.6 (DAI)
- net at U105.6 (DAI): now also U104.4 (DAO); no longer U106.4 (DAO)
- net at U76.3 (CLI): now also U75.1 (CLO); no longer U77.1 (CLO)
- net at U76.6 (DAI): now also U75.4 (DAO); no longer U77.4 (DAO)
- net at U346.1 (CLO): now also U347.3 (CLI); no longer U345.3 (CLI)
- net at U346.3 (CLI): now also U345.1 (CLO); no longer U347.1 (CLO)
- net at U346.4 (DAO): now also U347.6 (DAI); no longer U345.6 (DAI)
- net at U346.6 (DAI): now also U345.4 (DAO); no longer U347.4 (DAO)
- net at U344.1 (CLO): now also U345.3 (CLI); no longer U343.3 (CLI)
- net at U344.3 (CLI): now also U343.1 (CLO); no longer U345.1 (CLO)
- net at U344.4 (DAO): now also U345.6 (DAI); no longer U343.6 (DAI)
- net at U344.6 (DAI): now also U343.4 (DAO); no longer U345.4 (DAO)
- net at U388.1 (CLO): now also U389.3 (CLI); no longer U387.3 (CLI)
- net at U388.3 (CLI): now also U387.1 (CLO); no longer U389.1 (CLO)
- net at U388.4 (DAO): now also U389.6 (DAI); no longer U387.6 (DAI)
- net at U388.6 (DAI): now also U387.4 (DAO); no longer U389.4 (DAO)
- net at U319.1 (CLO): now also U320.3 (CLI); no longer U318.3 (CLI)
- net at U319.3 (CLI): now also U318.1 (CLO); no longer U320.1 (CLO)
- net at U319.4 (DAO): now also U320.6 (DAI); no longer U318.6 (DAI)
- net at U319.6 (DAI): now also U318.4 (DAO); no longer U320.4 (DAO)
- net at U401.1 (CLO): now also U402.3 (CLI); no longer U400.3 (CLI)
- net at U401.3 (CLI): now also U400.1 (CLO); no longer U402.1 (CLO)
- net at U401.4 (DAO): now also U402.6 (DAI); no longer U400.6 (DAI)
- net at U401.6 (DAI): now also U400.4 (DAO); no longer U402.4 (DAO)
- net at U349.1 (CLO): now also U350.3 (CLI); no longer U348.3 (CLI)
- net at U349.3 (CLI): now also U348.1 (CLO); no longer U350.1 (CLO)
- net at U349.4 (DAO): now also U350.6 (DAI); no longer U348.6 (DAI)
- net at U349.6 (DAI): now also U348.4 (DAO); no longer U350.4 (DAO)
- net at U144.1 (CLO): now also U145.3 (CLI); no longer U143.3 (CLI)
- net at U144.3 (CLI): now also U143.1 (CLO); no longer U145.1 (CLO)
- net at U144.4 (DAO): now also U145.6 (DAI); no longer U143.6 (DAI)
- net at U144.6 (DAI): now also U143.4 (DAO); no longer U145.4 (DAO)
- net at U43.3 (CLI): now also U42.1 (CLO); no longer U23.1 (CLO)
- net at U43.6 (DAI): now also U42.4 (DAO); no longer U23.4 (DAO)
- net at U70.1 (CLO): now also U71.3 (CLI); no longer U69.3 (CLI)
- net at U70.3 (CLI): now also U69.1 (CLO); no longer U71.1 (CLO)
- net at U70.4 (DAO): now also U71.6 (DAI); no longer U69.6 (DAI)
- net at U70.6 (DAI): now also U69.4 (DAO); no longer U71.4 (DAO)
- net at U243.3 (CLI): now also U242.1 (CLO); no longer U223.1 (CLO)
- net at U243.6 (DAI): now also U242.4 (DAO); no longer U223.4 (DAO)
- net at U357.1 (CLO): now also U358.3 (CLI); no longer U356.3 (CLI)
- net at U357.3 (CLI): now also U356.1 (CLO); no longer U358.1 (CLO)
- net at U357.4 (DAO): now also U358.6 (DAI); no longer U356.6 (DAI)
- net at U357.6 (DAI): now also U356.4 (DAO); no longer U358.4 (DAO)
- net at U351.1 (CLO): now also U352.3 (CLI); no longer U350.3 (CLI)
- net at U351.3 (CLI): now also U350.1 (CLO); no longer U352.1 (CLO)
- net at U351.4 (DAO): now also U352.6 (DAI); no longer U350.6 (DAI)
- net at U351.6 (DAI): now also U350.4 (DAO); no longer U352.4 (DAO)
- net at U398.1 (CLO): now also U399.3 (CLI); no longer U397.3 (CLI)
- net at U398.4 (DAO): now also U399.6 (DAI); no longer U397.6 (DAI)
- net at U196.1 (CLO): now also U197.3 (CLI); no longer U195.3 (CLI)
- net at U196.3 (CLI): now also U195.1 (CLO); no longer U197.1 (CLO)
- net at U196.4 (DAO): now also U197.6 (DAI); no longer U195.6 (DAI)
- net at U196.6 (DAI): now also U195.4 (DAO); no longer U197.4 (DAO)
- net at U303.3 (CLI): now also U302.1 (CLO); no longer U304.1 (CLO)
- net at U303.6 (DAI): now also U302.4 (DAO); no longer U304.4 (DAO)
- net at U262.1 (CLO): now also U263.3 (CLI); no longer U282.3 (CLI)
- net at U262.4 (DAO): now also U263.6 (DAI); no longer U282.6 (DAI)
- net at U202.1 (CLO): no longer U201.3 (CLI)
- net at U202.3 (CLI): now also U201.1 (CLO); no longer U182.1 (CLO)
- net at U202.4 (DAO): no longer U201.6 (DAI)
- net at U202.6 (DAI): now also U201.4 (DAO); no longer U182.4 (DAO)
- net at U200.1 (CLO): now also U201.3 (CLI); no longer U199.3 (CLI)
- net at U200.3 (CLI): now also U199.1 (CLO); no longer U201.1 (CLO)
- net at U200.4 (DAO): now also U201.6 (DAI); no longer U199.6 (DAI)
- net at U200.6 (DAI): now also U199.4 (DAO); no longer U201.4 (DAO)
- net at U66.1 (CLO): now also U67.3 (CLI); no longer U65.3 (CLI)
- net at U66.3 (CLI): now also U65.1 (CLO); no longer U67.1 (CLO)
- net at U66.4 (DAO): now also U67.6 (DAI); no longer U65.6 (DAI)
- net at U66.6 (DAI): now also U65.4 (DAO); no longer U67.4 (DAO)
- net at U109.1 (CLO): now also U110.3 (CLI); no longer U108.3 (CLI)
- net at U109.3 (CLI): now also U108.1 (CLO); no longer U110.1 (CLO)
- net at U109.4 (DAO): now also U110.6 (DAI); no longer U108.6 (DAI)
- net at U109.6 (DAI): now also U108.4 (DAO); no longer U110.4 (DAO)
- net at U31.1 (CLO): now also U32.3 (CLI); no longer U30.3 (CLI)
- net at U31.4 (DAO): now also U32.6 (DAI); no longer U30.6 (DAI)
- net at U35.1 (CLO): now also U36.3 (CLI); no longer U34.3 (CLI)
- net at U35.3 (CLI): now also U34.1 (CLO); no longer U36.1 (CLO)
- net at U35.4 (DAO): now also U36.6 (DAI); no longer U34.6 (DAI)
- net at U35.6 (DAI): now also U34.4 (DAO); no longer U36.4 (DAO)
- net at U359.1 (CLO): now also U360.3 (CLI); no longer U358.3 (CLI)
- net at U359.4 (DAO): now also U360.6 (DAI); no longer U358.6 (DAI)
- net at U119.1 (CLO): now also U120.3 (CLI); no longer U118.3 (CLI)
- net at U119.3 (CLI): now also U118.1 (CLO); no longer U120.1 (CLO)
- net at U119.4 (DAO): now also U120.6 (DAI); no longer U118.6 (DAI)
- net at U119.6 (DAI): now also U118.4 (DAO); no longer U120.4 (DAO)
- net at U363.3 (CLI): now also U362.1 (CLO); no longer U343.1 (CLO)
- net at U363.6 (DAI): now also U362.4 (DAO); no longer U343.4 (DAO)
- net at U146.1 (CLO): now also U147.3 (CLI); no longer U145.3 (CLI)
- net at U146.3 (CLI): now also U145.1 (CLO); no longer U147.1 (CLO)
- net at U146.4 (DAO): now also U147.6 (DAI); no longer U145.6 (DAI)
- net at U146.6 (DAI): now also U145.4 (DAO); no longer U147.4 (DAO)
- net at U353.1 (CLO): now also U354.3 (CLI); no longer U352.3 (CLI)
- net at U353.4 (DAO): now also U354.6 (DAI); no longer U352.6 (DAI)
- net at U276.1 (CLO): now also U277.3 (CLI); no longer U275.3 (CLI)
- net at U276.3 (CLI): now also U275.1 (CLO); no longer U277.1 (CLO)
- net at U276.4 (DAO): now also U277.6 (DAI); no longer U275.6 (DAI)
- net at U276.6 (DAI): now also U275.4 (DAO); no longer U277.4 (DAO)
- net at U398.3 (CLI): now also U397.1 (CLO); no longer U399.1 (CLO)
- net at U398.6 (DAI): now also U397.4 (DAO); no longer U399.4 (DAO)
- net at U74.1 (CLO): now also U75.3 (CLI); no longer U73.3 (CLI)
- net at U74.3 (CLI): now also U73.1 (CLO); no longer U75.1 (CLO)
- net at U74.4 (DAO): now also U75.6 (DAI); no longer U73.6 (DAI)
- net at U74.6 (DAI): now also U73.4 (DAO); no longer U75.4 (DAO)
- net at U385.1 (CLO): now also U386.3 (CLI); no longer U384.3 (CLI)
- net at U385.3 (CLI): now also U384.1 (CLO); no longer U386.1 (CLO)
- net at U385.4 (DAO): now also U386.6 (DAI); no longer U384.6 (DAI)
- net at U385.6 (DAI): now also U384.4 (DAO); no longer U386.4 (DAO)
- net at U111.1 (CLO): now also U112.3 (CLI); no longer U110.3 (CLI)
- net at U111.4 (DAO): now also U112.6 (DAI); no longer U110.6 (DAI)
- net at U234.1 (CLO): now also U235.3 (CLI); no longer U233.3 (CLI)
- net at U234.4 (DAO): now also U235.6 (DAI); no longer U233.6 (DAI)
- net at U265.1 (CLO): now also U266.3 (CLI); no longer U264.3 (CLI)
- net at U265.3 (CLI): now also U264.1 (CLO); no longer U266.1 (CLO)
- net at U265.4 (DAO): now also U266.6 (DAI); no longer U264.6 (DAI)
- net at U265.6 (DAI): now also U264.4 (DAO); no longer U266.4 (DAO)
- net at U154.1 (CLO): now also U155.3 (CLI); no longer U153.3 (CLI)
- net at U154.3 (CLI): now also U153.1 (CLO); no longer U155.1 (CLO)
- net at U154.4 (DAO): now also U155.6 (DAI); no longer U153.6 (DAI)
- net at U154.6 (DAI): now also U153.4 (DAO); no longer U155.4 (DAO)
- net at U263.1 (CLO): now also U264.3 (CLI); no longer U283.3 (CLI)
- net at U263.4 (DAO): now also U264.6 (DAI); no longer U283.6 (DAI)
- net at U316.1 (CLO): now also U317.3 (CLI); no longer U315.3 (CLI)
- net at U316.3 (CLI): now also U315.1 (CLO); no longer U317.1 (CLO)
- net at U316.4 (DAO): now also U317.6 (DAI); no longer U315.6 (DAI)
- net at U316.6 (DAI): now also U315.4 (DAO); no longer U317.4 (DAO)
- net at U152.3 (CLI): now also U151.1 (CLO); no longer U153.1 (CLO)
- net at U152.6 (DAI): now also U151.4 (DAO); no longer U153.4 (DAO)
- net at U359.3 (CLI): now also U358.1 (CLO); no longer U360.1 (CLO)
- net at U361.1 (CLO): now also U362.3 (CLI); no longer U360.3 (CLI)
- net at U359.6 (DAI): now also U358.4 (DAO); no longer U360.4 (DAO)
- net at U361.4 (DAO): now also U362.6 (DAI); no longer U360.6 (DAI)
- net at U240.1 (CLO): now also U241.3 (CLI); no longer U239.3 (CLI)
- net at U240.3 (CLI): now also U239.1 (CLO); no longer U241.1 (CLO)
- net at U240.4 (DAO): now also U241.6 (DAI); no longer U239.6 (DAI)
- net at U240.6 (DAI): now also U239.4 (DAO); no longer U241.4 (DAO)
- net at U123.3 (CLI): now also U122.1 (CLO); no longer U103.1 (CLO)
- net at U123.6 (DAI): now also U122.4 (DAO); no longer U103.4 (DAO)
- net at U194.3 (CLI): now also U193.1 (CLO); no longer U195.1 (CLO)
- net at U194.6 (DAI): now also U193.4 (DAO); no longer U195.4 (DAO)
- net at U185.3 (CLI): now also U184.1 (CLO); no longer U186.1 (CLO)
- net at U185.6 (DAI): now also U184.4 (DAO); no longer U186.4 (DAO)
- net at U64.3 (CLI): now also U63.1 (CLO); no longer U65.1 (CLO)
- net at U64.6 (DAI): now also U63.4 (DAO); no longer U65.4 (DAO)
- net at U342.1 (CLO): now also U343.3 (CLI); no longer U362.3 (CLI)
- net at U342.4 (DAO): now also U343.6 (DAI); no longer U362.6 (DAI)
- net at U268.1 (CLO): now also U269.3 (CLI); no longer U267.3 (CLI)
- net at U268.3 (CLI): now also U267.1 (CLO); no longer U269.1 (CLO)
- net at U268.4 (DAO): now also U269.6 (DAI); no longer U267.6 (DAI)
- net at U268.6 (DAI): now also U267.4 (DAO); no longer U269.4 (DAO)
- net at U355.1 (CLO): now also U356.3 (CLI); no longer U354.3 (CLI)
- net at U355.3 (CLI): now also U354.1 (CLO); no longer U356.1 (CLO)
- net at U355.4 (DAO): now also U356.6 (DAI); no longer U354.6 (DAI)
- net at U355.6 (DAI): now also U354.4 (DAO); no longer U356.4 (DAO)
- net at U230.1 (CLO): now also U231.3 (CLI); no longer U229.3 (CLI)
- net at U230.4 (DAO): now also U231.6 (DAI); no longer U229.6 (DAI)
- net at U234.3 (CLI): now also U233.1 (CLO); no longer U235.1 (CLO)
- net at U234.6 (DAI): now also U233.4 (DAO); no longer U235.4 (DAO)
- net at U26.1 (CLO): now also U27.3 (CLI); no longer U25.3 (CLI)
- net at U26.3 (CLI): now also U25.1 (CLO); no longer U27.1 (CLO)
- net at U26.4 (DAO): now also U27.6 (DAI); no longer U25.6 (DAI)
- net at U26.6 (DAI): now also U25.4 (DAO); no longer U27.4 (DAO)
- net at U280.1 (CLO): now also U281.3 (CLI); no longer U279.3 (CLI)
- net at U280.3 (CLI): now also U279.1 (CLO); no longer U281.1 (CLO)
- net at U280.4 (DAO): now also U281.6 (DAI); no longer U279.6 (DAI)
- net at U280.6 (DAI): now also U279.4 (DAO); no longer U281.4 (DAO)
- net at U230.3 (CLI): now also U229.1 (CLO); no longer U231.1 (CLO)
- net at U230.6 (DAI): now also U229.4 (DAO); no longer U231.4 (DAO)
- net at U41.3 (CLI): now also U40.1 (CLO); no longer U42.1 (CLO)
- net at U42.3 (CLI): now also U41.1 (CLO); no longer U22.1 (CLO)
- net at U41.6 (DAI): now also U40.4 (DAO); no longer U42.4 (DAO)
- net at U42.6 (DAI): now also U41.4 (DAO); no longer U22.4 (DAO)
- net at U156.1 (CLO): now also U157.3 (CLI); no longer U155.3 (CLI)
- net at U156.4 (DAO): now also U157.6 (DAI); no longer U155.6 (DAI)
- net at U303.1 (CLO): now also U304.3 (CLI); no longer U323.3 (CLI)
- net at U303.4 (DAO): now also U304.6 (DAI); no longer U323.6 (DAI)
- net at U238.3 (CLI): now also U237.1 (CLO); no longer U239.1 (CLO)
- net at U238.6 (DAI): now also U237.4 (DAO); no longer U239.4 (DAO)
- net at U313.1 (CLO): now also U314.3 (CLI); no longer U312.3 (CLI)
- net at U313.3 (CLI): now also U312.1 (CLO); no longer U314.1 (CLO)
- net at U313.4 (DAO): now also U314.6 (DAI); no longer U312.6 (DAI)
- net at U313.6 (DAI): now also U312.4 (DAO); no longer U314.4 (DAO)
- net at U223.3 (CLI): now also U222.1 (CLO); no longer U224.1 (CLO)
- net at U223.6 (DAI): now also U222.4 (DAO); no longer U224.4 (DAO)
- net at U163.3 (CLI): now also U162.1 (CLO); no longer U143.1 (CLO)
- net at U163.6 (DAI): now also U162.4 (DAO); no longer U143.4 (DAO)
- net at U31.3 (CLI): now also U30.1 (CLO); no longer U32.1 (CLO)
- net at U33.1 (CLO): now also U34.3 (CLI); no longer U32.3 (CLI)
- net at U31.6 (DAI): now also U30.4 (DAO); no longer U32.4 (DAO)
- net at U33.4 (DAO): now also U34.6 (DAI); no longer U32.6 (DAI)
- net at U103.3 (CLI): now also U102.1 (CLO); no longer U104.1 (CLO)
- net at U103.6 (DAI): now also U102.4 (DAO); no longer U104.4 (DAO)
- net at U278.3 (CLI): now also U277.1 (CLO); no longer U279.1 (CLO)
- net at U278.6 (DAI): now also U277.4 (DAO); no longer U279.4 (DAO)
- net at U68.1 (CLO): now also U69.3 (CLI); no longer U67.3 (CLI)
- net at U68.4 (DAO): now also U69.6 (DAI); no longer U67.6 (DAI)
- net at U353.3 (CLI): now also U352.1 (CLO); no longer U354.1 (CLO)
- net at U353.6 (DAI): now also U352.4 (DAO); no longer U354.4 (DAO)
- net at U272.1 (CLO): now also U273.3 (CLI); no longer U271.3 (CLI)
- net at U272.3 (CLI): now also U271.1 (CLO); no longer U273.1 (CLO)
- net at U272.4 (DAO): now also U273.6 (DAI); no longer U271.6 (DAI)
- net at U272.6 (DAI): now also U271.4 (DAO); no longer U273.4 (DAO)
- net at U278.1 (CLO): now also U279.3 (CLI); no longer U277.3 (CLI)
- net at U278.4 (DAO): now also U279.6 (DAI); no longer U277.6 (DAI)
- net at U76.1 (CLO): now also U77.3 (CLI); no longer U75.3 (CLI)
- net at U76.4 (DAO): now also U77.6 (DAI); no longer U75.6 (DAI)
- net at U83.3 (CLI): now also U82.1 (CLO); no longer U63.1 (CLO)
- net at U83.6 (DAI): now also U82.4 (DAO); no longer U63.4 (DAO)
- net at U68.3 (CLI): now also U67.1 (CLO); no longer U69.1 (CLO)
- net at U68.6 (DAI): now also U67.4 (DAO); no longer U69.4 (DAO)
- net at U189.1 (CLO): now also U190.3 (CLI); no longer U188.3 (CLI)
- net at U189.4 (DAO): now also U190.6 (DAI); no longer U188.6 (DAI)
- net at U72.1 (CLO): now also U73.3 (CLI); no longer U71.3 (CLI)
- net at U72.4 (DAO): now also U73.6 (DAI); no longer U71.6 (DAI)
- net at U39.3 (CLI): now also U38.1 (CLO); no longer U40.1 (CLO)
- net at U40.3 (CLI): now also U39.1 (CLO); no longer U41.1 (CLO)
- net at U39.6 (DAI): now also U38.4 (DAO); no longer U40.4 (DAO)
- net at U40.6 (DAI): now also U39.4 (DAO); no longer U41.4 (DAO)
- net at U394.1 (CLO): now also U395.3 (CLI); no longer U393.3 (CLI)
- net at U394.3 (CLI): now also U393.1 (CLO); no longer U395.1 (CLO)
- net at U394.4 (DAO): now also U395.6 (DAI); no longer U393.6 (DAI)
- net at U394.6 (DAI): now also U393.4 (DAO); no longer U395.4 (DAO)
- net at U191.1 (CLO): now also U192.3 (CLI); no longer U190.3 (CLI)
- net at U191.3 (CLI): now also U190.1 (CLO); no longer U192.1 (CLO)
- net at U191.4 (DAO): now also U192.6 (DAI); no longer U190.6 (DAI)
- net at U191.6 (DAI): now also U190.4 (DAO); no longer U192.4 (DAO)
- net at U282.1 (CLO): now also U283.3 (CLI); no longer U281.3 (CLI)
- net at U282.4 (DAO): now also U283.6 (DAI); no longer U281.6 (DAI)
- net at U122.3 (CLI): now also U121.1 (CLO); no longer U102.1 (CLO)
- net at U122.6 (DAI): now also U121.4 (DAO); no longer U102.4 (DAO)
- net at U72.3 (CLI): now also U71.1 (CLO); no longer U73.1 (CLO)
- net at U72.6 (DAI): now also U71.4 (DAO); no longer U73.4 (DAO)
- net at U270.1 (CLO): now also U271.3 (CLI); no longer U269.3 (CLI)
- net at U270.3 (CLI): now also U269.1 (CLO); no longer U271.1 (CLO)
- net at U270.4 (DAO): now also U271.6 (DAI); no longer U269.6 (DAI)
- net at U270.6 (DAI): now also U269.4 (DAO); no longer U271.4 (DAO)
- net at U64.1 (CLO): now also U65.3 (CLI); no longer U63.3 (CLI)
- net at U64.4 (DAO): now also U65.6 (DAI); no longer U63.6 (DAI)
- net at U236.1 (CLO): now also U237.3 (CLI); no longer U235.3 (CLI)
- net at U236.3 (CLI): now also U235.1 (CLO); no longer U237.1 (CLO)
- net at U236.4 (DAO): now also U237.6 (DAI); no longer U235.6 (DAI)
- net at U236.6 (DAI): now also U235.4 (DAO); no longer U237.4 (DAO)
- net at U117.1 (CLO): now also U118.3 (CLI); no longer U116.3 (CLI)
- net at U117.3 (CLI): now also U116.1 (CLO); no longer U118.1 (CLO)
- net at U117.4 (DAO): now also U118.6 (DAI); no longer U116.6 (DAI)
- net at U117.6 (DAI): now also U116.4 (DAO); no longer U118.4 (DAO)
- net at U238.1 (CLO): now also U239.3 (CLI); no longer U237.3 (CLI)
- net at U238.4 (DAO): now also U239.6 (DAI); no longer U237.6 (DAI)
- net at U189.3 (CLI): now also U188.1 (CLO); no longer U190.1 (CLO)
- net at U189.6 (DAI): now also U188.4 (DAO); no longer U190.4 (DAO)
- net at U111.3 (CLI): now also U110.1 (CLO); no longer U112.1 (CLO)
- net at U113.1 (CLO): now also U114.3 (CLI); no longer U112.3 (CLI)
- net at U111.6 (DAI): now also U110.4 (DAO); no longer U112.4 (DAO)
- net at U113.4 (DAO): now also U114.6 (DAI); no longer U112.6 (DAI)
- net at U194.1 (CLO): now also U195.3 (CLI); no longer U193.3 (CLI)
- net at U194.4 (DAO): now also U195.6 (DAI); no longer U193.6 (DAI)
- net at U37.1 (CLO): now also U38.3 (CLI); no longer U36.3 (CLI)
- net at U37.3 (CLI): now also U36.1 (CLO); no longer U38.1 (CLO)
- net at U37.4 (DAO): now also U38.6 (DAI); no longer U36.6 (DAI)
- net at U37.6 (DAI): now also U36.4 (DAO); no longer U38.4 (DAO)
- net at U33.3 (CLI): now also U32.1 (CLO); no longer U34.1 (CLO)
- net at U33.6 (DAI): now also U32.4 (DAO); no longer U34.4 (DAO)
- net at U274.1 (CLO): now also U275.3 (CLI); no longer U273.3 (CLI)
- net at U274.3 (CLI): now also U273.1 (CLO); no longer U275.1 (CLO)
- net at U274.4 (DAO): now also U275.6 (DAI); no longer U273.6 (DAI)
- net at U274.6 (DAI): now also U273.4 (DAO); no longer U275.4 (DAO)
- net at U150.3 (CLI): now also U149.1 (CLO); no longer U151.1 (CLO)
- net at U152.1 (CLO): now also U153.3 (CLI); no longer U151.3 (CLI)
- net at U150.6 (DAI): now also U149.4 (DAO); no longer U151.4 (DAO)
- net at U152.4 (DAO): now also U153.6 (DAI); no longer U151.6 (DAI)
- net at U311.1 (CLO): now also U312.3 (CLI); no longer U310.3 (CLI)
- net at U311.3 (CLI): now also U310.1 (CLO); no longer U312.1 (CLO)
- net at U311.4 (DAO): now also U312.6 (DAI); no longer U310.6 (DAI)
- net at U311.6 (DAI): now also U310.4 (DAO); no longer U312.4 (DAO)
- net at U185.1 (CLO): now also U186.3 (CLI); no longer U184.3 (CLI)
- net at U185.4 (DAO): now also U186.6 (DAI); no longer U184.6 (DAI)
- net at U307.1 (CLO): now also U308.3 (CLI); no longer U306.3 (CLI)
- net at U307.4 (DAO): now also U308.6 (DAI); no longer U306.6 (DAI)
- net at U161.1 (CLO): now also U162.3 (CLI); no longer U160.3 (CLI)
- net at U161.3 (CLI): now also U160.1 (CLO); no longer U162.1 (CLO)
- net at U161.4 (DAO): now also U162.6 (DAI); no longer U160.6 (DAI)
- net at U161.6 (DAI): now also U160.4 (DAO); no longer U162.4 (DAO)
- net at U309.3 (CLI): now also U308.1 (CLO); no longer U310.1 (CLO)
- net at U309.6 (DAI): now also U308.4 (DAO); no longer U310.4 (DAO)
- net at U107.3 (CLI): now also U106.1 (CLO); no longer U108.1 (CLO)
- net at U107.6 (DAI): now also U106.4 (DAO); no longer U108.4 (DAO)
- net at U198.1 (CLO): now also U199.3 (CLI); no longer U197.3 (CLI)
- net at U198.4 (DAO): now also U199.6 (DAI); no longer U197.6 (DAI)
- net at U307.3 (CLI): now also U306.1 (CLO); no longer U308.1 (CLO)
- net at U307.6 (DAI): now also U306.4 (DAO); no longer U308.4 (DAO)
- net at U121.3 (CLI): now also U120.1 (CLO); no longer U122.1 (CLO)
- net at U121.6 (DAI): now also U120.4 (DAO); no longer U122.4 (DAO)
- net at U23.3 (CLI): now also U22.1 (CLO); no longer U24.1 (CLO)
- net at U23.6 (DAI): now also U22.4 (DAO); no longer U24.4 (DAO)
- net at U107.1 (CLO): now also U108.3 (CLI); no longer U106.3 (CLI)
- net at U107.4 (DAO): now also U108.6 (DAI); no longer U106.6 (DAI)
- net at U183.1 (CLO): now also U184.3 (CLI)
- net at U183.3 (CLI): now also U182.1 (CLO); no longer U184.1 (CLO)
- net at U183.4 (DAO): now also U184.6 (DAI)
- net at U183.6 (DAI): now also U182.4 (DAO); no longer U184.4 (DAO)
- net at U113.3 (CLI): now also U112.1 (CLO); no longer U114.1 (CLO)
- net at U113.6 (DAI): now also U112.4 (DAO); no longer U114.4 (DAO)
- net at U158.1 (CLO): now also U159.3 (CLI); no longer U157.3 (CLI)
- net at U158.3 (CLI): now also U157.1 (CLO); no longer U159.1 (CLO)
- net at U158.4 (DAO): now also U159.6 (DAI); no longer U157.6 (DAI)
- net at U158.6 (DAI): now also U157.4 (DAO); no longer U159.4 (DAO)
- net at U309.1 (CLO): now also U310.3 (CLI); no longer U308.3 (CLI)
- net at U309.4 (DAO): now also U310.6 (DAI); no longer U308.6 (DAI)
- net at U198.3 (CLI): now also U197.1 (CLO); no longer U199.1 (CLO)
- net at U198.6 (DAI): now also U197.4 (DAO); no longer U199.4 (DAO)
- net at U156.3 (CLI): now also U155.1 (CLO); no longer U157.1 (CLO)
- net at U156.6 (DAI): now also U155.4 (DAO); no longer U157.4 (DAO)
- net at U142.1 (CLO): now also U143.3 (CLI); no longer U162.3 (CLI)
- net at U142.4 (DAO): now also U143.6 (DAI); no longer U162.6 (DAI)
- net at U361.3 (CLI): now also U360.1 (CLO); no longer U362.1 (CLO)
- net at U361.6 (DAI): now also U360.4 (DAO); no longer U362.4 (DAO)
- net at U115.1 (CLO): now also U116.3 (CLI); no longer U114.3 (CLI)
- net at U115.4 (DAO): now also U116.6 (DAI); no longer U114.6 (DAI)
- net at U24.3 (CLI): now also U23.1 (CLO); no longer U25.1 (CLO)
- net at U24.6 (DAI): now also U23.4 (DAO); no longer U25.4 (DAO)
- net at U148.1 (CLO): now also U149.3 (CLI); no longer U147.3 (CLI)
- net at U148.4 (DAO): now also U149.6 (DAI); no longer U147.6 (DAI)
- net at U115.3 (CLI): now also U114.1 (CLO); no longer U116.1 (CLO)
- net at U115.6 (DAI): now also U114.4 (DAO); no longer U116.4 (DAO)
- net at U242.3 (CLI): now also U241.1 (CLO); no longer U222.1 (CLO)
- net at U242.6 (DAI): now also U241.4 (DAO); no longer U222.4 (DAO)
- net at U148.3 (CLI): now also U147.1 (CLO); no longer U149.1 (CLO)
- net at U148.6 (DAI): now also U147.4 (DAO); no longer U149.4 (DAO)
- net at U150.1 (CLO): now also U151.3 (CLI); no longer U149.3 (CLI)
- net at U150.4 (DAO): now also U151.6 (DAI); no longer U149.6 (DAI)
- new net: U226.1 (CLO), U227.3 (CLI)
- new net: U226.4 (DAO), U227.6 (DAI)
- new net: U399.1 (CLO), U400.3 (CLI)
- new net: U399.4 (DAO), U400.6 (DAI)
- new net: U389.1 (CLO), U390.3 (CLI)
- new net: U389.4 (DAO), U390.6 (DAI)
- new net: U347.1 (CLO), U348.3 (CLI)
- new net: U347.4 (DAO), U348.6 (DAI)
- new net: U314.1 (CLO), U315.3 (CLI)
- new net: U314.4 (DAO), U315.6 (DAI)
- new net: U223.1 (CLO), U224.3 (CLI)
- new net: U223.4 (DAO), U224.6 (DAI)
- new net: U103.1 (CLO), U104.3 (CLI)
- new net: U103.4 (DAO), U104.6 (DAI)
- new net: U27.1 (CLO), U28.3 (CLI)
- new net: U27.4 (DAO), U28.6 (DAI)
- new net: U320.1 (CLO), U321.3 (CLI)
- new net: U320.4 (DAO), U321.6 (DAI)
- new net: U386.1 (CLO), U387.3 (CLI)
- new net: U386.4 (DAO), U387.6 (DAI)
- new net: U281.1 (CLO), U282.3 (CLI)
- new net: U281.4 (DAO), U282.6 (DAI)
- new net: U392.1 (CLO), U393.3 (CLI)
- new net: U392.4 (DAO), U393.6 (DAI)
- new net: U266.1 (CLO), U267.3 (CLI)
- new net: U266.4 (DAO), U267.6 (DAI)
- new net: U79.1 (CLO), U80.3 (CLI)
- new net: U79.4 (DAO), U80.6 (DAI)
- new net: U317.1 (CLO), U318.3 (CLI)
- new net: U317.4 (DAO), U318.6 (DAI)
- new net: U192.1 (CLO), U193.3 (CLI)
- new net: U192.4 (DAO), U193.6 (DAI)
- new net: U24.1 (CLO), U25.3 (CLI)
- new net: U24.4 (DAO), U25.6 (DAI)
- new net: U159.1 (CLO), U160.3 (CLI)
- new net: U159.4 (DAO), U160.6 (DAI)
Other:
- moved on the sheet: U103, U104, U105, U106, U107, U108, U109, U110, U111, U112, U113, U114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

Commit message: Added led connections on pcb
Connections:
- no-connect marks 28 -> 32

Commit message: +feat: finished second pcb design
Parts:
- removed JT1: ~, LED_SMD:UART JT, symbol LED:UART_JT
- added LED_CON1, LED_CON2: ~, RF_Module:led_con, symbol Connector:led_con
- added pwr1, pwr2: ~, RF_Module:5vgnd, symbol Connector:5vgnd
- added rxtx1: ~, RF_Module:rxtx, symbol Connector:rxtx
Connections:
- net +5V: now also pwr1.1 (5v), pwr2.1 (5v)
- net GND: now also pwr1.2 (gnd), pwr2.2 (gnd)
- net UART_RX: now also rxtx1.1 (rx)
- net UART_TX: now also rxtx1.2 (tx)
- net at U2.15 (IO3), U203.3 (CLI): now also LED_CON2.1 (cli)
- net at U2.4 (IO4), U203.6 (DAI): now also LED_CON2.2 (dai)
- net at U2.38 (IO2), U3.6 (DAI): now also LED_CON1.2 (dai)
- net at U2.39 (IO1), U3.3 (CLI): now also LED_CON1.1 (cli)
